File: ez80.kicad_sch (KiCad schematic)
At the start: 57 parts, among them Q1 ASE-18.432MHZ-L-C-T, U3 EZ80F92AZ020EG(LQFP100), U4 AS7C34096A-10TCTR

Commit message: schematics finished, pcb routing 80%
Parts:
- removed BUF1, BUF2: SN74LVC1G125DBVR, OLIMEX_IC-FP:SOT-23-5, symbol AgonLight2_Rev_B:SN74LVC1G125DBVR
- removed BUF3: SN74LVC1G04DBVR(SOT23-5), OLIMEX_IC-FP:SOT-23-5, symbol AgonLight2_Rev_B:SN74LVC1G04DBVR(SOT23-5)
- removed C10, C20, C21, C22, C23, C7, C8, C9: 100nF/10V/20%/X5R/0402, OLIMEX_RLC-FP:C_0402_5MIL_DWS, symbol AgonLight2_Rev_B:C
- removed C11, C12, C13, C14, C16, C17, C18, C19: 1nF/X7R/50VDC/0402, OLIMEX_RLC-FP:C_0402_5MIL_DWS, symbol AgonLight2_Rev_B:C
- removed C24, C25, C26, C27, C3, C4, C5, C6: 10uF/6.3V/20%/X5R/0603, OLIMEX_RLC-FP:C_0603_5MIL_DWS, symbol AgonLight2_Rev_B:C
- removed Q1: ASE-18.432MHZ-L-C-T, OLIMEX_Crystal-FP:Oscillator-18.432MHz-3.2x2.5mm, symbol AgonLight2_Rev_B:Oscillator-100MHZ_TXC-7W
- removed R42, R43, R44, R45, R46, R47, R51: 33R/0603, OLIMEX_RLC-FP:R_0603_5MIL_DWS, symbol AgonLight2_Rev_B:R
- removed R49, R50, R52: 4.7K/0603, OLIMEX_RLC-FP:R_0603_5MIL_DWS, symbol AgonLight2_Rev_B:R
- removed U3: EZ80F92AZ020EG(LQFP100), OLIMEX_IC-FP:LQFP-100_14x14mm_STM32H730VBT6, symbol AgonLight2_Rev_B:EZ80F92AZ020SG(LQFP100)
- removed UART_DIS1: HN1x2+MJ6, OLIMEX_Jumpers-FP:HN1x2_Jumper, symbol AgonLight2_Rev_B:JP1E
- added BT1: Battery_Cell, Connector_PinHeader_2.54mm:PinHeader_1x02_P2.54mm_Vertical, symbol Device:Battery_Cell
- added C1, C2: 22pF, HexAgonFootprintsLibrary:C_0402_5MIL_DWS, symbol AgonLight2_Rev_B:C
- added C33: 18pF, HexAgonFootprintsLibrary:C_0402_5MIL_DWS, symbol AgonLight2_Rev_B:C
- added C34: 100nF/10V/20%/X5R/0402, HexAgonFootprintsLibrary:C_0402_5MIL_DWS, symbol AgonLight2_Rev_B:C
- added C35: 56nF, HexAgonFootprintsLibrary:C_0402_5MIL_DWS, symbol AgonLight2_Rev_B:C
- added C36: 270pF, HexAgonFootprintsLibrary:C_0402_5MIL_DWS, symbol AgonLight2_Rev_B:C
- added C38, C39, C40, C41, C42, C43, C44, C45, C46, C47, C48, C49, C51, C52, C53, C54, C55, C56, C57, C58, C59, C60, C61, C62, C63, C64: 1nF/X7R/50VDC/0402, HexAgonFootprintsLibrary:C_0402_5MIL_DWS, symbol AgonLight2_Rev_B:C
- added C50: 10uF/6.3V/20%/X5R/0603, HexAgonFootprintsLibrary:C_0603_5MIL_DWS, symbol AgonLight2_Rev_B:C
- added D3: 1N5819S4/SOD123, HexAgonFootprintsLibrary:SOD-123_1C-2A_KA, symbol AgonLight2_Rev_B:D_Schottky
- added J2: Conn_02x40_Top_Bottom, Connector_PinHeader_2.54mm:PinHeader_2x40_P2.54mm_Vertical, symbol Connector_Generic:Conn_02x40_Top_Bottom
- added R1, R23, R35, R37, R59, R60, R62, R63, R64, R65, R67, R68, R69, R70, R74, R75, R80: 33R/0603, HexAgonFootprintsLibrary:R_0603_5MIL_DWS, symbol AgonLight2_Rev_B:R
- added R38: 10K/0603, HexAgonFootprintsLibrary:R_0603_5MIL_DWS, symbol AgonLight2_Rev_B:R
- added R61: 100K/0603, HexAgonFootprintsLibrary:R_0603_5MIL_DWS, symbol AgonLight2_Rev_B:R
- added R66: 499R/0603, HexAgonFootprintsLibrary:R_0603_5MIL_DWS, symbol AgonLight2_Rev_B:R
- added U1, U10, U11, U13, U15, U16, U17: SN74LVC245APW, Package_SO:TSSOP-24_4.4x7.8mm_P0.65mm, symbol HexAgonLib:SN74LVC8T245
- added U5: ~, Package_QFP:LQFP-144-1EP_20x20mm_P0.5mm_EP6.5x6.5mm, symbol HexAgonLib:ez80f91
- added Y1: 5Mhz, Crystal:Crystal_SMD_Abracon_ABM3-2Pin_5.0x3.2mm, symbol Device:Crystal
- added Y2: 32.768kHz, Crystal:Crystal_SMD_Abracon_ABM3-2Pin_5.0x3.2mm, symbol Device:Crystal
- C15: value 100nF/10V/20%/X5R/0402 -> 18pF; footprint OLIMEX_RLC-FP:C_0402_5MIL_DWS -> HexAgonFootprintsLibrary:C_0402_5MIL_DWS
- C28: value 100nF/10V/20%/X5R/0402 -> 1nF/X7R/50VDC/0402; footprint OLIMEX_RLC-FP:C_0402_5MIL_DWS -> HexAgonFootprintsLibrary:C_0402_5MIL_DWS
- C29, C32: footprint OLIMEX_RLC-FP:C_0603_5MIL_DWS -> HexAgonFootprintsLibrary:C_0603_5MIL_DWS
- C30, C31: footprint OLIMEX_RLC-FP:C_0402_5MIL_DWS -> HexAgonFootprintsLibrary:C_0402_5MIL_DWS
- R39, R40, R41, R48, R58: footprint OLIMEX_RLC-FP:R_0603_5MIL_DWS -> HexAgonFootprintsLibrary:R_0603_5MIL_DWS
- R53: value 4.7K/0603 -> 2.2K/0603; footprint OLIMEX_RLC-FP:R_0603_5MIL_DWS -> HexAgonFootprintsLibrary:R_0603_5MIL_DWS
- R54, R55: value 4.7K/0603 -> 10K/0603; footprint OLIMEX_RLC-FP:R_0603_5MIL_DWS -> HexAgonFootprintsLibrary:R_0603_5MIL_DWS
- R56: value 10K/0603 -> 33R/0603; footprint OLIMEX_RLC-FP:R_0603_5MIL_DWS -> HexAgonFootprintsLibrary:R_0603_5MIL_DWS
- R57: value 33R/0603 -> 10K/0603; footprint OLIMEX_RLC-FP:R_0603_5MIL_DWS -> HexAgonFootprintsLibrary:R_0603_5MIL_DWS
- U4: footprint OLIMEX_IC-FP:TSOP-44_Pitch-0.80mm_18.80x11.80x1.20mm -> HexAgonFootprintsLibrary:TSOP-44_Pitch-0.80mm_18.80x11.80x1.20mm
Connections:
- net +3.3V: now also C28.2, C38.2, C39.2, C40.2, C41.2, C42.2, C43.2, C44.2, C45.2, C46.2, C47.2, C48.2, C49.2, C50.2, C51.2, C54.2, C56.2, C58.2, C60.2, C62.2, C63.2, D3.1 (K), R38.1, U1.1 (V_{CCA}), U10.23 (V_{CCB}), U10.24 (V_{CCB}), U11.23 (V_{CCB}), U11.24 (V_{CCB}), U13.23 (V_{CCB}), U13.24 (V_{CCB}), U15.23 (V_{CCB}), U15.24 (V_{CCB}), U16.23 (V_{CCB}), U16.24 (V_{CCB}), U17.1 (V_{CCA}), U5.112 (Vdd), U5.122 (Vdd), U5.133 (Vdd), U5.14 (Vdd), U5.22 (Vdd), U5.31 (Vdd), U5.37 (Vdd), U5.47 (Vdd), U5.59 (Vdd), U5.6 (Vdd), U5.63 (RTC_Vdd), U5.81 (Vdd), U5.87 (PLL_Vdd), U5.88 (Vdd), U5.98 (Vdd); no longer C28.1, R56.2
- net GND: now also C28.1, BT1.2 (-), C1.2, C2.2, C33.2, C34.2, C35.2, C36.1, C38.1, C39.1, C40.1, C41.1, C42.1, C43.1, C44.1, C45.1, C46.1, C47.1, C48.1, C49.1, C50.1, C51.1, C52.1, C53.1, C54.1, C55.1, C56.1, C57.1, C58.1, C59.1, C60.1, C61.1, C62.1, C63.1, C64.1, J2.17 (Pin_17), J2.57 (Pin_57), U1.10 (A8), U1.11 (GND), U1.12 (GND), U1.13 (GND), U1.14 (B8), U1.15 (B7), U1.16 (B6), U1.17 (B5), U1.18 (B4), U1.2 (DIR), U1.22 (~{OE}), U1.6 (A4), U1.7 (A5), U1.8 (A6), U1.9 (A7), U10.11 (GND), U10.12 (GND), U10.13 (GND), U10.2 (DIR), U10.22 (~{OE}), U11.11 (GND), U11.12 (GND), U11.13 (GND), U11.2 (DIR), U11.22 (~{OE}), U13.11 (GND), U13.12 (GND), U13.13 (GND), U13.2 (DIR), U13.22 (~{OE}), U15.11 (GND), U15.12 (GND), U15.13 (GND), U15.18 (B4), U15.19 (B3), U15.2 (DIR), U15.20 (B2), U15.21 (B1), U15.22 (~{OE}), U15.3 (A1), U15.4 (A2), U15.5 (A3), U15.6 (A4), U16.11 (GND), U16.12 (GND), U16.13 (GND), U16.2 (DIR), U16.22 (~{OE}), U17.11 (GND), U17.12 (GND), U17.13 (GND), U17.22 (~{OE}), U5.108 (Vss), U5.113 (Vss), U5.123 (Vss), U5.134 (Vss), U5.15 (Vss), U5.23 (Vss), U5.32 (Vss), U5.38 (Vss), U5.48 (Vss), U5.60 (Vss), U5.64 (Vss), U5.7 (Vss), U5.72 (Vss), U5.82 (Vss), U5.84 (PLL_Vss), U5.89 (Vss), U5.99 (Vss); no longer C28.2
- net EZ80_RTS: now reaches R56.1
- net ~{CS2}: now reaches R39.2
- net ~{CS2}: now also U15.15 (B7)
- net at R48.2: now also U5.71 (~{TRST})
- net ~{CS3}: now reaches R40.2
- net ~{CS3}: now also U15.14 (B8)
- net INT: now reaches R57.2
- net INT: now also J2.22 (Pin_22)
- net at R41.2: now also U5.66 (TMS)
- net ~{CS0}: now reaches R58.2
- net ~{CS0}: now also U4.8 (~{CE})
- net BUF1 renamed +5Vrc
- net +5Vrc: now also C52.2, C53.2, C55.2, C57.2, C59.2, C61.2, C64.2, J2.18 (Pin_18), J2.58 (Pin_58), U1.23 (V_{CCB}), U1.24 (V_{CCB}), U10.1 (V_{CCA}), U11.1 (V_{CCA}), U13.1 (V_{CCA}), U15.1 (V_{CCA}), U16.1 (V_{CCA}), U17.23 (V_{CCB}), U17.24 (V_{CCB})
- net CS renamed ~{WAIT}
- net ~{WAIT}: now also U1.5 (A3), U5.54 (~{WAIT}); no longer U4.8 (~{CE})
- net ESP_RXD: no longer names the net of R58.1
- net ESP_RXD: now also U5.33 (~{CS0})
- removed net RD: R39.1, R54.2, U4.37 (~{OE})
- net RST\EN: no longer names the net of C15.1
- net RST\EN: now also R60.2, R61.1, Y1.2
- net SRAM_A0 renamed A0
- net A0: now also U10.14 (B8), U5.1 (A0)
- net SRAM_A1 renamed A1
- net A1: now also U10.15 (B7), U5.2 (A1)
- net SRAM_A10 renamed A11
- net A11: now also U11.17 (B5), U5.16 (A11)
- net SRAM_A11 renamed A10
- net A10: now also U11.16 (B6), U5.13 (A10)
- net SRAM_A12 renamed A12
- net A12: now also U11.18 (B4), U5.17 (A12)
- net SRAM_A13 renamed A13
- net A13: now also U11.19 (B3), U5.18 (A13)
- net SRAM_A14 renamed A14
- net A14: now also U11.20 (B2), U5.19 (A14)
- net SRAM_A15 renamed A15
- net A15: now also U11.21 (B1), U5.20 (A15)
- net SRAM_A16 renamed A16
- net A16: now also U13.14 (B8), U5.21 (A16)
- net SRAM_A17 renamed A17
- net A17: now also U13.15 (B7), U5.24 (A17)
- net SRAM_A18 renamed A18
- net A18: now also U13.16 (B6), U5.25 (A18)
- net SRAM_A2 renamed A2
- net A2: now also U10.16 (B6), U5.3 (A2)
- net SRAM_A3 renamed A3
- net A3: now also U10.17 (B5), U5.4 (A3)
- net SRAM_A4 renamed A4
- net A4: now also U10.18 (B4), U5.5 (A4)
- net SRAM_A5 renamed A5
- net A5: now also U10.19 (B3), U5.8 (A5)
- net SRAM_A6 renamed A6
- net A6: now also U10.20 (B2), U5.9 (A6)
- net SRAM_A7 renamed A7
- net A7: now also U10.21 (B1), U5.10 (A7)
- net SRAM_A8 renamed A8
- net A8: now also U11.14 (B8), U5.11 (A8)
- net SRAM_A9 renamed A9
- net A9: now also U11.15 (B7), U5.12 (A9)
- net SRAM_DATA0 renamed DATA0
- net DATA0: now also U17.3 (A1), U5.39 (DATA0)
- net SRAM_DATA1 renamed DATA1
- net DATA1: now also U17.4 (A2), U5.40 (DATA1)
- net SRAM_DATA2 renamed DATA2
- net DATA2: now also U17.5 (A3), U5.41 (DATA2)
- net SRAM_DATA3 renamed DATA3
- net DATA3: now also U17.6 (A4), U5.42 (DATA3)
- net SRAM_DATA4 renamed DATA4
- net DATA4: now also U17.7 (A5), U5.43 (DATA4)
- net SRAM_DATA5 renamed DATA5
- net DATA5: now also U17.8 (A6), U5.44 (DATA5)
- net SRAM_DATA6 renamed DATA6
- net DATA6: now also U17.9 (A7), U5.45 (DATA6)
- net SRAM_DATA7 renamed DATA7
- net DATA7: now also U17.10 (A8), U5.46 (DATA7)
- removed net WR: R40.1, R55.2, U4.15 (~{WE})
- new net: R69.2, U5.107 (PB7)
- new net: C33.1, R61.2, U5.86 (Xin), Y1.1
- new net: R37.1, U5.58 (~{BUSACK})
- new net: R75.2, U5.110 (SCL)
- new net: R68.2, U5.103 (PB3)
- new net: C35.1, R66.2
- new net: R74.2, U5.109 (SDA)
- new net: C36.2, R66.1, U5.83 (LOOP_FILT)
- new net: R56.2, U5.75 (PD2)
- new net: R1.1, U5.49 (~{IORQ})
- new net: R70.2, U5.104 (PB4)
- new net: R63.1, U5.51 (~{RD})
- new net: R67.2, U5.102 (PB2)
- new net: R23.1, U5.111 (PHI)
- new net: R62.1, U5.34 (~{CS1})
- new net: R39.1, U5.35 (~{CS2})
- new net: R40.1, U5.36 (~{CS3})
- new net: R35.1, U5.50 (~{MREQ})
- new net: R64.1, U5.52 (~{WR})
- new net: R80.1, U5.53 (~{INSTRD})
- new net: C1.1, U5.61 (RTC_Xin), Y2.1
- new net: C2.1, U5.62 (RTC_Xout), Y2.2
- new net: R65.1, U5.65 (~{HALT_SLP})
- new net: R59.2, U5.73 (PD0)
- new net: R60.1, U5.85 (Xout)
- new net: BT1.1 (+), D3.2 (A)
- new net A19: U13.17 (B5), U5.26 (A19)
- new net A20: U13.18 (B4), U5.27 (A20)
- new net A21: U13.19 (B3), U5.28 (A21)
- new net A22: U13.20 (B2), U5.29 (A22)
- new net A23: U13.21 (B1), U5.30 (A23)
- new net D10: J2.69 (Pin_69)
- new net D11: J2.70 (Pin_70)
- new net D12: J2.71 (Pin_71)
- new net D13: J2.72 (Pin_72)
- new net D14: J2.73 (Pin_73)
- new net D15: J2.74 (Pin_74)
- new net EZ80_CTS: U5.76 (PD3)
- new net EZ80_INT_GENERAL: U5.100 (PB0)
- new net EZ80_INT_VSYNC: U5.101 (PB1)
- new net EZ80_MISO: U5.106 (PB6)
- new net EZ80_MOSI: R69.1
- new net EZ80_RxD: U5.74 (PD1)
- new net EZ80_SCK: R68.1
- new net EZ80_SCL: R75.1
- new net EZ80_SDA: R74.1
- new net EZ80_SS_ESP32: R67.1
- new net EZ80_SS_SD: R70.1
- new net EZ80_SYSCLK: R23.2, U16.16 (B6)
- new net EZ80_TCK: U5.67 (TCK)
- new net EZ80_TDI: U5.69 (TDI)
- new net EZ80_TxD: R59.1
- new net PA0: U5.114 (PA0)
- new net PA1: U5.115 (PA1)
- new net PA2: U5.116 (PA2)
- new net PA3: U5.117 (PA3)
- new net PA4: U5.118 (PA4)
- new net PA5: U5.119 (PA5)
- new net PA6: U5.120 (PA6)
- new net PA7: U5.121 (PA7)
- new net PB5: U5.105 (PB5)
- new net PC0: U5.90 (PC0)
- new net PC1: U5.91 (PC1)
- new net PC2: U5.92 (PC2)
- new net PC3: U5.93 (PC3)
- new net PC4: U5.94 (PC4)
- new net PC5: U5.95 (PC5)
- new net PC6: U5.96 (PC6)
- new net PC7: U5.97 (PC7)
- new net PD4: U5.77 (PD4)
- new net PD5: U5.78 (PD5)
- new net PD6: U5.79 (PD6)
- new net PD7: U5.80 (PD7)
- new net RX: J2.36 (Pin_36)
- new net RX2: J2.76 (Pin_76)
- new net TX: J2.35 (Pin_35)
- new net TX2: J2.75 (Pin_75)
- new net USER1: J2.37 (Pin_37)
- new net USER2: J2.38 (Pin_38)
- new net USER3: J2.39 (Pin_39)
- new net USER4: J2.40 (Pin_40)
- new net USER5: J2.77 (Pin_77)
- new net USER6: J2.78 (Pin_78)
- new net USER7: J2.79 (Pin_79)
- new net USER8: J2.80 (Pin_80)
- new net rcA0: J2.16 (Pin_16), U10.10 (A8)
- new net rcA1: J2.15 (Pin_15), U10.9 (A7)
- new net rcA10: J2.6 (Pin_6), U11.8 (A6)
- new net rcA11: J2.5 (Pin_5), U11.7 (A5)
- new net rcA12: J2.4 (Pin_4), U11.6 (A4)
- new net rcA13: J2.3 (Pin_3), U11.5 (A3)
- new net rcA14: J2.2 (Pin_2), U11.4 (A2)
- new net rcA15: J2.1 (Pin_1), U11.3 (A1)
- new net rcA16: J2.56 (Pin_56), U13.10 (A8)
- new net rcA17: J2.55 (Pin_55), U13.9 (A7)
- new net rcA18: J2.54 (Pin_54), U13.8 (A6)
- new net rcA19: J2.53 (Pin_53), U13.7 (A5)
- new net rcA2: J2.14 (Pin_14), U10.8 (A6)
- new net rcA20: J2.52 (Pin_52), U13.6 (A4)
- new net rcA21: J2.51 (Pin_51), U13.5 (A3)
- new net rcA22: J2.50 (Pin_50), U13.4 (A2)
- new net rcA23: J2.49 (Pin_49), U13.3 (A1)
- new net rcA3: J2.13 (Pin_13), U10.7 (A5)
- new net rcA4: J2.12 (Pin_12), U10.6 (A4)
- new net rcA5: J2.11 (Pin_11), U10.5 (A3)
- new net rcA6: J2.10 (Pin_10), U10.4 (A2)
- new net rcA7: J2.9 (Pin_9), U10.3 (A1)
- new net rcA8: J2.8 (Pin_8), U11.10 (A8)
- new net rcA9: J2.7 (Pin_7), U11.9 (A7)
- new net rcCLOCK: J2.21 (Pin_21), U16.8 (A6)
- new net rcCLOCK2: J2.61 (Pin_61)
- new net rcD0: J2.27 (Pin_27), U17.21 (B1)
- new net rcD1: J2.28 (Pin_28), U17.20 (B2)
- new net rcD2: J2.29 (Pin_29), U17.19 (B3)
- new net rcD3: J2.30 (Pin_30), U17.18 (B4)
- new net rcD4: J2.31 (Pin_31), U17.17 (B5)
- new net rcD5: J2.32 (Pin_32), U17.16 (B6)
- new net rcD6: J2.33 (Pin_33), U17.15 (B7)
- new net rcD7: J2.34 (Pin_34), U17.14 (B8)
- new net rcPAGE: J2.60 (Pin_60)
- new net ~{BUSACK}: R37.2, U16.15 (B7)
- new net ~{BUSREQ}: R38.2, U1.4 (A2), U5.57 (~{BUSREQ})
- new net ~{CS1}: R62.2, U15.16 (B6)
- new net ~{EZ80_RESET}: C34.1, U16.17 (B5), U5.55 (~{RESET})
- new net ~{HALT}: R65.2, U16.14 (B8)
- new net ~{IORQ}: R1.2, U16.19 (B3)
- new net ~{M1}: R80.2, U15.17 (B5)
- new net ~{MREQ}: R35.2, U16.18 (B4)
- new net ~{NMI}: R54.2, U1.3 (A1), U5.56 (~{NMI})
- new net ~{RD}: R63.2, U16.20 (B2), U17.2 (DIR), U4.37 (~{OE})
- new net ~{WP}: R55.2, U5.144 (~{WP})
- new net ~{WR}: R64.2, U16.21 (B1), U4.15 (~{WE})
- new net ~{rcBUSACK}: J2.62 (Pin_62), U16.9 (A7)
- new net ~{rcBUSREQ}: J2.64 (Pin_64), U1.20 (B2)
- new net ~{rcCS1}: J2.67 (Pin_67), U15.8 (A6)
- new net ~{rcCS2}: J2.68 (Pin_68), U15.9 (A7)
- new net ~{rcCS3}: U15.10 (A8)
- new net ~{rcHALT}: J2.63 (Pin_63), U16.10 (A8)
- new net ~{rcIORQ}: J2.26 (Pin_26), U16.5 (A3)
- new net ~{rcM1}: J2.19 (Pin_19), U15.7 (A5)
- new net ~{rcMREQ}: J2.23 (Pin_23), U16.6 (A4)
- new net ~{rcNMI}: J2.66 (Pin_66), U1.21 (B1)
- new net ~{rcRD}: J2.25 (Pin_25), U16.4 (A2)
- new net ~{rcRESET}: J2.20 (Pin_20), U16.7 (A5)
- new net ~{rcRFSH}: J2.59 (Pin_59)
- new net ~{rcWAIT}: J2.65 (Pin_65), U1.19 (B3)
- new net ~{rcWR}: J2.24 (Pin_24), U16.3 (A1)
- no-connect marks 15 -> 50
Other:
- note added: "continuous input from rcBus"
- note added: "continuous output to rcBus"
- note added: "~{RD}=H"
- note added: "~{RD}=L"
- moved on the sheet: C29, C30, C31, C32, R53, R54, U4

Commit message: 1st production and BOM
Parts:
- BT1: MfgNumber (none) -> 9-146276-0
- C1, C2: MfgNumber (none) -> GRM1555C1H220JA01J
- C15, C33: MfgNumber (none) -> GRM1555C1H180JA01D
- C28, C38, C39, C40, C41, C42, C43, C44, C45, C46, C47, C48, C49, C51, C52, C53, C54, C55, C56, C57, C58, C59, C60, C61, C62, C63, C64: MfgNumber (none) -> GRM155R61A102KA01D
- C29, C32, C50: MfgNumber (none) -> GRM185R60J106ME15J
- C30, C31, C34: MfgNumber (none) -> GRM022R61A104KE01L
- C35: MfgNumber (none) -> GRM155R71A563MA01J
- C36: MfgNumber (none) -> GRM155R71H271KA01J
- D3: MfgNumber (none) -> 1N5819HW-7-F
- J2: footprint Connector_PinHeader_2.54mm:PinHeader_2x40_P2.54mm_Vertical -> HexAgonFootprintsLibrary:PinHeader_2x40_P2.54mm_Vertical; MfgNumber (none) -> 9-146276-0
- R1, R23, R35, R37, R39, R40, R56, R58, R59, R60, R62, R63, R64, R65, R67, R68, R69, R70, R74, R75, R80: MfgNumber (none) -> ESR03EZPJ330
- R38, R54, R55, R57: MfgNumber (none) -> ESR03EZPJ103
- R41, R48: MfgNumber (none) -> ESR03EZPJ472
- R53: MfgNumber (none) -> ESR03EZPJ222
- R61: MfgNumber (none) -> ESR03EZPJ104
- R66: value 499R/0603 -> 499R/1%/0603; MfgNumber (none) -> ERJ-UP6F4990V
- U1, U10, U11, U13, U15, U16, U17: value SN74LVC245APW -> SN74LVC8T245; MfgNumber (none) -> 595-SN74LVC8T245PWR
- U4: MfgNumber (none) -> AS7C34096A-10TCN
- U5: value ~ -> EZ80F91; footprint Package_QFP:LQFP-144-1EP_20x20mm_P0.5mm_EP6.5x6.5mm -> HexAgonFootprintsLibrary:LQFP-144-1EP_20x20mm_P0.5mm_EP6.5x6.5mm; MfgNumber (none) -> EZ80F91AZA50EK
- Y1: footprint Crystal:Crystal_SMD_Abracon_ABM3-2Pin_5.0x3.2mm -> Crystal:Crystal_SMD_HC49-SD; MfgNumber (none) -> ABLS-5.000MHZ-B2-T
- Y2: footprint Crystal:Crystal_SMD_Abracon_ABM3-2Pin_5.0x3.2mm -> Crystal:Crystal_C26-LF_D2.1mm_L6.5mm_Horizontal; MfgNumber (none) -> ab26t-32.768khz
