File: keyboard_usb.kicad_sch (KiCad schematic)
At the start: 0 parts

Commit message: schematics finished, pcb routing 80%
Parts:
- added BTN1: B3F-3150, HexAgonFootprintsLibrary:B3F-31XX, symbol AgonLight2_Rev_B:T1107A(6x3,8x2,5MM)
- added C26, C65: 22uF/6.3V/20%/X5R/C0603, HexAgonFootprintsLibrary:C_0603_5MIL_DWS, symbol AgonLight2_Rev_B:C
- added C27: 1uF/10V/20%/X5R/C0603, HexAgonFootprintsLibrary:C_0603_5MIL_DWS, symbol AgonLight2_Rev_B:C
- added C3, C4: 100nF/10V/20%/X5R/0402, HexAgonFootprintsLibrary:C_0402_5MIL_DWS, symbol AgonLight2_Rev_B:C
- added C66: 0.1uF/6.3V/20%/X5R/C0603, HexAgonFootprintsLibrary:C_0603_5MIL_DWS, symbol AgonLight2_Rev_B:C
- added D4, D5: 1N5819S4/SOD123, HexAgonFootprintsLibrary:SOD-123_1C-2A_KA, symbol AgonLight2_Rev_B:D_Schottky
- added FET1, FET2: BSS138(SOT23-3), HexAgonFootprintsLibrary:SOT23, symbol AgonLight2_Rev_B:N-MOS+DIOD
- added L2, L3, L4: FB0805/600R/2A, HexAgonFootprintsLibrary:L_0805_5MIL_DWS, symbol AgonLight2_Rev_B:L
- added POWER1: LED/RED/0603, HexAgonFootprintsLibrary:LED_0603_KA, symbol AgonLight2_Rev_B:LED
- added Q4, Q5: BC817-40NPN(SOT23), HexAgonFootprintsLibrary:SOT23, symbol AgonLight2_Rev_B:Q_NPN_BEC
- added R18, R19, R83, R84: 5.1K/0603, HexAgonFootprintsLibrary:R_0603_5MIL_DWS, symbol AgonLight2_Rev_B:R
- added R42, R43, R52: 10K/0603, HexAgonFootprintsLibrary:R_0603_5MIL_DWS, symbol AgonLight2_Rev_B:R
- added R44, R45: NA(120R/0603), HexAgonFootprintsLibrary:R_0603_5MIL_DWS, symbol AgonLight2_Rev_B:R
- added R46, R47, R51, R82, R85: 2.2K/0603, HexAgonFootprintsLibrary:R_0603_5MIL_DWS, symbol AgonLight2_Rev_B:R
- added R86: 1k/0603, HexAgonFootprintsLibrary:R_0603_5MIL_DWS, symbol AgonLight2_Rev_B:R
- added U12: CP2102N-Axx-xQFN24, Package_DFN_QFN:QFN-24-1EP_4x4mm_P0.5mm_EP2.6x2.6mm, symbol Interface_USB:CP2102N-Axx-xQFN24
- added U14: TLV75533PDBV, Package_TO_SOT_SMD:SOT-23-5, symbol Regulator_Linear:TLV75533PDBV
- added U3: VDA2710NTA(SOT-23), HexAgonFootprintsLibrary:SOT-23, symbol AgonLight2_Rev_B:VDA2710NTA(SOT-23)
- added U7, U8: USBLC6-2P6, HexAgonFootprintsLibrary:SOT-666, symbol AgonLight2_Rev_B:USBLC6-2P6
- added USBA_KEYBOARD1: USB-SRWH-4A-LF(USB-A), HexAgonFootprintsLibrary:USB_PN87520_HOST_PTH, symbol AgonLight2_Rev_B:USB_A_MALE
- added USBC_OTG0, USBC_UART0: USB-C-16P-F(A40-00119-A52-12), HexAgonFootprintsLibrary:USB2.0_TYPE-C(A40-00119-A52-12), symbol AgonLight2_Rev_B:USB2.0_TYPE-C(A40-00119-A52-12)
Connections:
- new net: L3.1, USBC_UART0.0 (SHELL)
- new net: R83.1, USBC_UART0.A5 (CC1)
- new net: U7.3 (I/O2), USBC_UART0.A6 (DP1), USBC_UART0.B6 (DP2)
- new net: U7.1 (I/O1), USBC_UART0.A7 (DN1), USBC_UART0.B7 (DN2)
- new net: R84.1, USBC_UART0.B5 (CC2)
- new net: FET2.3 (D), R43.1, R45.1, USBA_KEYBOARD1.3 (D+)
- new net: FET1.3 (D), R42.1, R44.1, USBA_KEYBOARD1.2 (D-)
- new net: L2.1, USBA_KEYBOARD1.5 (SHIELD)
- new net: L4.1, USBC_OTG0.0 (SHELL)
- new net: R86.2, U12.9 (~{RST})
- new net: POWER1.1 (K), R51.1
- new net: R18.1, USBC_OTG0.A5 (CC1)
- new net: Q5.1 (B), R85.2
- new net: Q4.1 (B), R82.2
- new net: U8.3 (I/O2), USBC_OTG0.A6 (DP1), USBC_OTG0.B6 (DP2)
- new net: U8.1 (I/O1), USBC_OTG0.A7 (DN1), USBC_OTG0.B7 (DN2)
- new net: R19.1, USBC_OTG0.B5 (CC2)
- new net +3.3V: C26.1, C3.1, C65.1, C66.1, FET1.1 (G), FET2.1 (G), R46.2, R47.2, R52.2, R86.1, U12.5 (VIO), U12.6 (VDD), U12.7 (VREGIN), U14.5 (OUT), U3.3 (VIn)
- new net +5V_USB: C27.1, D4.1 (K), D5.1 (K), POWER1.2 (A), R42.2, R43.2, U12.8 (VBUS), U14.1 (IN), U14.3 (EN), USBA_KEYBOARD1.1 (VBUS)
- new net BOOT_MODE: Q5.3 (C)
- new net D+: U12.3 (D+), U7.4 (I/O2)
- new net D-: U12.4 (D-), U7.6 (I/O1)
- new net DTR: Q5.2 (E), R82.1, U12.23 (~{DTR})
- new net GND: BTN1.1, C26.2, C27.2, C3.2, C4.1, C65.2, C66.2, L2.2, L3.2, L4.2, R18.2, R19.2, R51.2, R83.2, R84.2, U12.2 (GND), U12.25 (GND), U14.2 (GND), U3.2 (Vss), U7.2 (GND), U8.2 (GND), USBA_KEYBOARD1.4 (GND), USBC_OTG0.A1 (GND), USBC_OTG0.A12 (GND), USBC_OTG0.B1 (GND), USBC_OTG0.B12 (GND), USBC_UART0.A1 (GND), USBC_UART0.A12 (GND), USBC_UART0.B1 (GND), USBC_UART0.B12 (GND)
- new net HOST_RXD: U12.20 (RXD)
- new net HOST_TXD: U12.21 (TXD)
- new net KCLK: FET2.2 (S), R45.2, R47.1
- new net KDAT: FET1.2 (S), R44.2, R46.1
- new net RTS: Q4.2 (E), R85.1, U12.19 (~{RTS})
- new net USB_OTG_D+: U8.4 (I/O2)
- new net USB_OTG_D-: U8.6 (I/O1)
- new net VBUS1: D5.2 (A), U7.5 (VBUS), USBC_UART0.A4 (VBUS), USBC_UART0.A9 (VBUS), USBC_UART0.B4 (VBUS), USBC_UART0.B9 (VBUS)
- new net VBUS2: D4.2 (A), U8.5 (VBUS), USBC_OTG0.A4 (VBUS), USBC_OTG0.A9 (VBUS), USBC_OTG0.B4 (VBUS), USBC_OTG0.B9 (VBUS)
- new net ~{RESET}: BTN1.2, C4.2, Q4.3 (C), R52.1, U3.1 (VOut)
- no-connect marks 0 -> 14

Commit message: 1st production and BOM
Parts:
- BTN1: MfgNumber (none) -> B3F-3150
- C26, C65: Fieldname 1 Value 1 -> (none); MfgNumber (none) -> GRM188R60J226MEA0D
- C27: Fieldname 1 Value 1 -> (none); MfgNumber (none) -> GRM188R61A105KA61J
- C3, C4: Fieldname 1 Value 1 -> (none); MfgNumber (none) -> GRM022R61A104KE01L
- C66: Fieldname 1 Value 1 -> (none); MfgNumber (none) -> GRM188R72A104MA35D
- D4, D5: MfgNumber (none) -> 1N5819HW-7-F
- FET1, FET2: MfgNumber (none) -> BSS138
- L2, L3, L4: MfgNumber (none) -> ILHB0805ER601V
- POWER1: Fieldname 1 Value 1 -> (none); MfgNumber (none) -> KS EELP41.22-P1R2-58-A8J8-020-R18
- Q4, Q5: MfgNumber (none) -> BC817K-25
- R18, R19, R83, R84: MfgNumber (none) -> ESR03EZPJ512
- R42, R43, R52: MfgNumber (none) -> ESR03EZPJ103
- R44, R45: MfgNumber (none) -> ESR03EZPJ121
- R46, R47: MfgNumber (none) -> ESR03EZPJ222
- R51, R82, R85: Fieldname 1 Value 1 -> (none); MfgNumber (none) -> ESR03EZPJ222
- R86: Fieldname 1 Value 1 -> (none); MfgNumber (none) -> ESR03EZPJ102
- U12: MfgNumber (none) -> CP2102N-A02-GQFN24R
- U14: MfgNumber (none) -> TLV75533PDBVR
- U3: MfgNumber (none) -> TLV803EB26RDBZR
- U7, U8: MfgNumber (none) -> USBLC6-2P6
- USBA_KEYBOARD1: MfgNumber (none) -> 292303-4
- USBC_OTG0, USBC_UART0: MfgNumber (none) -> USB4105-GF-A
