File: HexAgon.kicad_pcb (KiCad board)
At the start: 4 copper layers, 160 x 102.8 mm, 191 parts, among them J1 HEADER_3, J2 Conn_02x40_Top_Bottom, J3 Conn_02x16_Odd_Even, Q4 BC817-40NPN(SOT23), Q5 BC817-40NPN(SOT23), U1 SN74LVC245APW, U10 SN74LVC245APW, U11 SN74LVC245APW, U12 CP2102N-Axx-xQFN24, U13 SN74LVC245APW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

Commit message: v1.0 version PCB
Parts:
- added REF**: OSHW-Logo2_7.3x6mm_SilkScreen, Symbol:OSHW-Logo2_7.3x6mm_SilkScreen, F.Cu at (134.6, 76.8)
- J2: footprint Connector_PinHeader_2.54mm:PinHeader_2x40_P2.54mm_Vertical -> HexAgonFootprintsLibrary:PinHeader_2x40_P2.54mm_Vertical
- U5: footprint Package_QFP:LQFP-144-1EP_20x20mm_P0.5mm_EP6.5x6.5mm -> HexAgonFootprintsLibrary:LQFP-144-1EP_20x20mm_P0.5mm_EP6.5x6.5mm
- moved R51 36.5 mm to (223.6, 142.0), turned to 90 degrees
- moved POWER1 35.8 mm to (221.6, 142.0), turned to 90 degrees
- moved L3 12.7 mm to (226.8, 93.2)
- moved C27 12.4 mm to (222.6, 110.7), turned to -90 degrees
- moved D4 11.7 mm to (229.9, 109.8)
- moved D5 11.7 mm to (229.9, 105.2)
- moved C26 9.37 mm to (219.1, 113.9), turned to 0 degrees
- moved U14 7.70 mm to (219.2, 110.7), turned to 180 degrees
- moved L2 7.23 mm to (143.8, 55.6), turned to -90 degrees
- moved C35 6.26 mm to (171.3, 104.4), turned to -90 degrees
- moved ZDI1 5.00 mm to (173.4, 119.2)
- moved L4 4.55 mm to (226.6, 122.0)
- moved C36 4.12 mm to (166.3, 104.4)
- moved C22 3.84 mm to (180.2, 138.2)
- moved C18 3.81 mm to (177.8, 138.2)
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Routing:
- net GND: track 544.8 -> 326.8 mm, vias 84 -> 102
- net /EZ80 ports/EZ80_SDA: track 22.6 -> 148.5 mm, vias 0 -> 5
- net /EZ80 ports/EZ80_SCL: track 22.7 -> 147.5 mm, vias 0 -> 5
- net /EZ80/PC0: track 0.00 -> 109.3 mm, vias 0 -> 4
- net /EZ80/CLOCK: track 47.7 -> 155.6 mm, vias 2 -> 7
- net /EZ80 ports/GPIO_B5: track 0.00 -> 95.0 mm, vias 0 -> 4
- net /EZ80/PC7: track 0.00 -> 92.3 mm, vias 0 -> 4
- net /EZ80/PC5: track 0.00 -> 90.2 mm, vias 0 -> 4
- net /ESP32/ESP_SPI_MISO: track 147.8 -> 236.3 mm, vias 7 -> 11
- net /EZ80/PC6: track 0.00 -> 88.2 mm, vias 0 -> 4
- net /EZ80/PC3: track 0.00 -> 86.1 mm, vias 0 -> 4
- net /EZ80/PC4: track 0.00 -> 85.0 mm, vias 0 -> 4
- net /EZ80 ports/EZ80_SS_SD: track 8.33 -> 92.1 mm, vias 0 -> 6
- net /EZ80/PC2: track 43.3 -> 113.5 mm, vias 0 -> 5
- net /EZ80/PC1: track 35.7 -> 100.0 mm, vias 0 -> 5
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- added copper zone on In2.Cu, net +5V_USB
- added copper zone on In2.Cu, net /ESP32 ports/VBUS1
- added copper zone on In2.Cu, net /ESP32 ports/VBUS2
Other:
- outline, holes or cut-outs redrawn
- board text added: "HexAgon v1.0 (c) 2025 - S0urceror"

Commit message: 1st production and BOM
Parts:
- removed REF**: OSHW-Logo2_7.3x6mm_SilkScreen, Symbol:OSHW-Logo2_7.3x6mm_SilkScreen
- C11, C12, C20, C21: value 100nF -> 0.1uF/6.3V/20%/X5R/C0603
- C25: value 22uF/6.3V/20%/X5R/0603 -> 22uF/6.3V/20%/X5R/C0603
- R66: value 499R/0603 -> 499R/1%/0603
- R71: value NA -> 100K/0603
- U1, U10, U11, U13, U15, U16, U17: value SN74LVC245APW -> SN74LVC8T245
- U5: value ~ -> EZ80F91
- Y1: footprint Crystal:Crystal_SMD_Abracon_ABM3-2Pin_5.0x3.2mm -> Crystal:Crystal_SMD_HC49-SD
- Y2: footprint Crystal:Crystal_SMD_Abracon_ABM3-2Pin_5.0x3.2mm -> Crystal:Crystal_C26-LF_D2.1mm_L6.5mm_Horizontal
- moved C1 7.95 mm to (158.6, 127.7)
- moved C2 7.47 mm to (158.6, 122.5), turned to 0 degrees
- moved C15 7.29 mm to (177.2, 104.7), turned to 90 degrees
- moved Y1 6.17 mm to (173.4, 100.9)
- moved C33 5.91 mm to (177.1, 97.2), turned to -90 degrees
- moved R61 3.48 mm to (169.7, 99.4)
- moved C35 2.14 mm to (169.6, 105.7), turned to 0 degrees
- moved R60 1.82 mm to (167.2, 102.1)
- moved Y2 1.47 mm to (153.4, 126.0), turned to 90 degrees
- moved R66 0.50 mm to (168.8, 104.0)
- moved C27 0.16 mm to (222.5, 110.8), turned to 90 degrees
Routing:
- net Net-(U5-RTC_Xin): track 16.9 -> 23.0 mm
- net Net-(C15-Pad1): track 8.00 -> 13.7 mm
- net GND: track 326.8 -> 330.3 mm
- net +5V_USB: track 292.6 -> 294.7 mm
- net Net-(U5-Xout): track 8.19 -> 6.57 mm
- net Net-(U5-RTC_Xout): track 19.3 -> 20.7 mm
- net /ESP32/ESP_INT_GENERAL: track 73.0 -> 74.0 mm
- net Net-(U5-Xin): track 18.7 -> 19.7 mm

Commit message: fixed SD card issues
Connections:
- GPIO1 pad 27: /ESP32/ESP_SPI_MOSI -> /ESP32/ESP_SPI_MISO
- GPIO1 pad 32: /ESP32/ESP_SPI_MISO -> /ESP32/ESP_SPI_MOSI
- MICRO_SD1 pad 3: /ESP32/ESP_SPI_MISO -> /ESP32/ESP_SPI_MOSI
- R69 pad 1: /ESP32/ESP_SPI_MISO -> /ESP32/ESP_SPI_MOSI
- R72 pad 1: /ESP32/ESP_SPI_MISO -> /ESP32/ESP_SPI_MOSI
- R73 pad 2: /ESP32/ESP_SPI_MOSI -> /ESP32/ESP_SPI_MISO
- R78 pad 1: /ESP32/ESP_SPI_MOSI -> /ESP32/ESP_SPI_MISO
- U5 pad 106: /ESP32/ESP_SPI_MOSI -> /ESP32/ESP_SPI_MISO
- UEXT1 pad 7: /ESP32/ESP_SPI_MOSI -> /ESP32/ESP_SPI_MISO
- UEXT1 pad 8: /ESP32/ESP_SPI_MISO -> /ESP32/ESP_SPI_MOSI
Routing:
- net /ESP32/ESP_SPI_MISO: track 236.3 -> 212.1 mm, vias 11 -> 8
- net /ESP32/ESP_SPI_MOSI: track 212.5 -> 236.3 mm, vias 10 -> 11
